File: hardware/OHBeacon/OHBeacon.kicad_pcb (KiCad board)
At the start: 2 copper layers, 90 x 65 mm, 33 parts, among them J1 Conn_01x01_Pin, J2 Conn_01x01_Pin, J3 Conn_01x01_Pin, J4 Conn_01x01_Pin, J5 USB_C_Receptacle_PowerOnly_6P, J6 Conn_01x04_Socket, P1 S2B-ZR-SM4A-TF, SW1 EN, SW2 I09, U1 ESP32-C3-WROOM-02

Commit message: get james approval
Parts:
- added C13: 10uF, Capacitor_SMD:C_0805_2012Metric_Pad1.18x1.45mm_HandSolder, F.Cu at (85.7, 103.5)
- added C14: 10uF, Capacitor_SMD:C_0805_2012Metric_Pad1.18x1.45mm_HandSolder, F.Cu at (85.7, 100.0)
- added C15: 1.0uF, Capacitor_SMD:C_0805_2012Metric_Pad1.18x1.45mm_HandSolder, F.Cu at (104.2, 99.0)
- added C16: 1.0uF, Capacitor_SMD:C_0805_2012Metric_Pad1.18x1.45mm_HandSolder, F.Cu at (104.2, 102.0)
- added C17: 0.1uF, Capacitor_SMD:C_0805_2012Metric_Pad1.18x1.45mm_HandSolder, F.Cu at (91.7, 91.5)
- added D10: RED, LED_SMD:LED_0805_2012Metric_Pad1.15x1.40mm_HandSolder, F.Cu at (104.2, 95.0)
- added D9: GREEN, LED_SMD:LED_0805_2012Metric_Pad1.15x1.40mm_HandSolder, F.Cu at (85.7, 95.0)
- added Q1: DMG2305UX-7, DMG2305UX-7:SOT91P240X110-3N_DMG2305UX-7, F.Cu at (97.5, 93.1)
- added R1: 1K, Resistor_SMD:R_0805_2012Metric_Pad1.20x1.40mm_HandSolder, F.Cu at (85.8, 91.5)
- added R5: 5k1, Resistor_SMD:R_0805_2012Metric_Pad1.20x1.40mm_HandSolder, F.Cu at (100.0, 106.5)
- added R6: 5k1, Resistor_SMD:R_0805_2012Metric_Pad1.20x1.40mm_HandSolder, F.Cu at (90.5, 106.5)
- added R7: 10k, Resistor_SMD:R_0805_2012Metric_Pad1.20x1.40mm_HandSolder, F.Cu at (95.2, 106.5)
- added R8: 1k, Resistor_SMD:R_0805_2012Metric_Pad1.20x1.40mm_HandSolder, F.Cu at (104.2, 91.5)
- added R9: 10k, Resistor_SMD:R_0805_2012Metric_Pad1.20x1.40mm_HandSolder, F.Cu at (91.8, 95.0)
- added U3: AP2112K-3.3, Package_TO_SOT_SMD:SOT-23-5, F.Cu at (98.9, 100.5)
- added U4: MCP73831-2-OT, Package_TO_SOT_SMD:SOT-23-5, F.Cu at (91.0, 100.8)
- moved J5 1.00 mm to (95.2, 113.0)
Connections:
- C1 pad 1: +BATT -> /BATT_VCC
- C2 pad 1: +BATT -> /BATT_VCC
- C3 pad 1: +BATT -> /BATT_VCC
- C4 pad 1: +BATT -> /BATT_VCC
- C5 pad 1: +BATT -> /BATT_VCC
- C6 pad 1: +BATT -> /BATT_VCC
- C7 pad 1: +BATT -> /BATT_VCC
- C8 pad 1: +BATT -> /BATT_VCC
- D1 pad 1: +BATT -> /BATT_VCC
- D2 pad 1: +BATT -> /BATT_VCC
- D3 pad 1: +BATT -> /BATT_VCC
- D4 pad 1: +BATT -> /BATT_VCC
- D5 pad 1: +BATT -> /BATT_VCC
- D6 pad 1: +BATT -> /BATT_VCC
- D7 pad 1: +BATT -> /BATT_VCC
- D8 pad 1: +BATT -> /BATT_VCC
- U1 pad 6: unconnected-(U1-IO7-Pad6) -> /IO7
