File: hardware/OHBeacon/OHBeacon.kicad_pcb (KiCad board)
At the start: 2 copper layers, 90 x 65 mm, 49 parts, among them J1 Conn_01x01_Pin, J2 Conn_01x01_Pin, J3 Conn_01x01_Pin, J4 Conn_01x01_Pin, J5 USB_C_Receptacle_PowerOnly_6P, J6 Conn_01x04_Socket, P1 S2B-ZR-SM4A-TF, Q1 DMG2305UX-7, SW1 EN, SW2 I09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

Commit message: final pcb?
Parts:
- removed C17: 0.1uF, Capacitor_SMD:C_0805_2012Metric_Pad1.18x1.45mm_HandSolder
- removed Q1: DMG2305UX-7, DMG2305UX-7:SOT91P240X110-3N_DMG2305UX-7
- removed R9: 10k, Resistor_SMD:R_0805_2012Metric_Pad1.20x1.40mm_HandSolder
- added Q2: AO3400A, Package_TO_SOT_SMD:SOT-23, F.Cu at (59.0, 68.1)
- added R10: 1M, Resistor_SMD:R_0805_2012Metric_Pad1.20x1.40mm_HandSolder, F.Cu at (118.9, 64.2)
- added R100: 100, Resistor_SMD:R_0805_2012Metric_Pad1.20x1.40mm_HandSolder, F.Cu at (58.5, 65.0)
- added R11: 1M, Resistor_SMD:R_0805_2012Metric_Pad1.20x1.40mm_HandSolder, F.Cu at (118.9, 66.4)
- added R12: 1M, Resistor_SMD:R_0805_2012Metric_Pad1.20x1.40mm_HandSolder, F.Cu at (118.9, 68.5)
- R7: value 10k -> 2k
- moved R8 16.4 mm to (88.7, 96.7), turned to -90 degrees
- moved C16 13.8 mm to (96.5, 90.6), turned to 180 degrees
- moved D10 12.4 mm to (91.8, 95.4)
- moved R7 9.56 mm to (91.8, 97.6), turned to 180 degrees
- moved U3 9.53 mm to (101.1, 91.3), turned to 180 degrees
- moved C13 8.57 mm to (94.0, 101.3), turned to 90 degrees
- moved C15 7.59 mm to (106.1, 91.6), turned to -90 degrees
- moved C14 2.23 mm to (87.0, 101.8), turned to 90 degrees
- moved D9 1.40 mm to (84.4, 94.5)
- moved R1 1.40 mm to (84.4, 91.0)
- moved D1 0.44 mm to (121.3, 55.9)
- moved U4 0.44 mm to (90.6, 100.6)
Connections:
- C1 pad 1: /BATT_VCC -> +BATT
- C1 pad 2: GND -> /LED_GND
- C2 pad 1: /BATT_VCC -> +BATT
- C2 pad 2: GND -> /LED_GND
- C3 pad 1: /BATT_VCC -> +BATT
- C3 pad 2: GND -> /LED_GND
- C4 pad 1: /BATT_VCC -> +BATT
- C4 pad 2: GND -> /LED_GND
- C5 pad 1: /BATT_VCC -> +BATT
- C5 pad 2: GND -> /LED_GND
- C6 pad 1: /BATT_VCC -> +BATT
- C6 pad 2: GND -> /LED_GND
- C7 pad 1: /BATT_VCC -> +BATT
- C7 pad 2: GND -> /LED_GND
- C8 pad 1: /BATT_VCC -> +BATT
- C8 pad 2: GND -> /LED_GND
- D1 pad 1: /BATT_VCC -> +BATT
- D1 pad 3: GND -> /LED_GND
- D2 pad 1: /BATT_VCC -> +BATT
- D2 pad 3: GND -> /LED_GND
- D3 pad 1: /BATT_VCC -> +BATT
- D3 pad 3: GND -> /LED_GND
- D4 pad 1: /BATT_VCC -> +BATT
- D4 pad 3: GND -> /LED_GND
- D5 pad 1: /BATT_VCC -> +BATT
- D5 pad 3: GND -> /LED_GND
- D6 pad 1: /BATT_VCC -> +BATT
- D6 pad 3: GND -> /LED_GND
- D7 pad 1: /BATT_VCC -> +BATT
- D7 pad 3: GND -> /LED_GND
- D8 pad 1: /BATT_VCC -> +BATT
- D8 pad 3: GND -> /LED_GND
- U1 pad 18: unconnected-(U1-IO0-Pad18) -> /ADC
Routing:
- net /LED_GND: track 0.00 -> 272.7 mm, vias 0 -> 12
- net +BATT: track 0.00 -> 261.4 mm, vias 0 -> 17
- net +5V: track 0.00 -> 133.2 mm, vias 0 -> 11
- net /EN: track 0.00 -> 53.8 mm
- net /DCON: track 0.00 -> 49.4 mm
- net GND: track 0.00 -> 49.3 mm, vias 0 -> 23
- net Net-(D7-DOUT): track 0.00 -> 46.6 mm
- net Net-(D5-DOUT): track 0.00 -> 44.9 mm
- net /IO9: track 0.00 -> 37.5 mm
- net Net-(D2-DOUT): track 0.00 -> 31.4 mm
- net /DIN: track 0.00 -> 27.9 mm
- net /IO7: track 0.00 -> 27.2 mm, vias 0 -> 2
- net Net-(D1-DOUT): track 0.00 -> 26.7 mm, vias 0 -> 2
- net Net-(D3-DOUT): track 0.00 -> 26.5 mm
- net /ADC: track 0.00 -> 19.1 mm, vias 0 -> 2
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- added copper zone on F.Cu, net +3.3V
- added copper zone on B.Cu, net +5V
- added copper zone on F.Cu, net +5V
- added copper zone on B.Cu, net +BATT
- added copper zone on F.Cu, net +BATT
- added copper zone on B.Cu, net GND
- added copper zone on F.Cu, net GND

Commit message: for aryan
Routing:
- net /EN: vias 0 -> 2
Changed lines of the file:
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@@
-	)
-	(segment
-		(start 82.42 57.31)
-		(end 83.48 58.37)
-		(width 0.5)
-		(layer "F.Cu")
-		(net 3)
 	)
 	(segment
@@
 		(start 93 81)
 		(end 92.5 80.5)
-		(width 0.5)
-		(layer "F.Cu")
-		(net 3)
-	)
-	(segment
-		(start 85.651 58.401)
-		(end 86.25 59)
 		(width 0.5)
 		(layer "F.Cu")
@@
 		(start 93 85.5)
 		(end 93 81)
+		(width 0.5)
+		(layer "F.Cu")
+		(net 3)
+	)
+	(segment
+		(start 82.42 57.31)
+		(end 82.56 57.31)
 		(width 0.5)
 		(layer "F.Cu")
@@
 	)
 	(segment
-		(start 83.48 58.37)
-		(end 83.48 58.401)
+		(start 82.24 57.3)
+		(end 82.25 57.31)
 		(width 0.5)
 		(layer "F.Cu")
@@
 	)
 	(segment
-		(start 82.24 57.3)
-		(end 82.25 57.31)
+		(start 82.56 57.31)
+		(end 82.75 57.5)
 		(width 0.5)
 		(layer "F.Cu")
@@
 	)
 	(segment
-		(start 83.48 58.401)
-		(end 85.651 58.401)
+		(start 85 59)
+		(end 86.25 59)
 		(width 0.5)
 		(layer "F.Cu")
 		(net 3)
 	)
+	(via
+		(at 85 59)
+		(size 0.6)
+		(drill 0.3)
+		(layers "F.Cu" "B.Cu")
+		(net 3)
+	)
+	(via
+		(at 82.75 57.5)
+		(size 0.6)
+		(drill 0.3)
+		(layers "F.Cu" "B.Cu")
+		(net 3)
+	)
+	(segment
+		(start 84.25 59)
+		(end 85 59)
+		(width 0.5)
+		(layer "B.Cu")
+		(net 3)
+	)
+	(segment
+		(start 82.75 57.5)
+		(end 84.25 59)
+		(width 0.5)
+		(layer "B.Cu")
+		(net 3)
+	)

Commit message: even more final PCB???
Parts:
- added R13: 500, Resistor_SMD:R_0805_2012Metric_Pad1.20x1.40mm_HandSolder, F.Cu at (114.6, 53.2)
- added R9: 100k, Resistor_SMD:R_0805_2012Metric_Pad1.20x1.40mm_HandSolder, F.Cu at (55.4, 68.0)
Connections:
- U1 pad 15: /DIN -> Net-(U1-IO3)
Routing:
- net /DIN: track 27.9 -> 11.7 mm
- net Net-(U1-IO3): track 0.00 -> 15.2 mm
- net Net-(Q2-G): track 2.36 -> 4.57 mm
- net GND: track 49.3 -> 51.5 mm
