File: hardware/OHBeacon/OHBeacon.kicad_sch (KiCad schematic)
At the start: 49 parts, among them J1 Conn_01x01_Pin, J2 Conn_01x01_Pin, J3 Conn_01x01_Pin, J4 Conn_01x01_Pin, J5 USB_C_Receptacle_PowerOnly_6P, J6 Conn_01x04_Socket, P1 S2B-ZR-SM4A-TF, Q1 DMG2305UX-7, SW1 EN, SW2 I09, U1 ESP32-C3-WROOM-02, U3 AP2112K-3.3, U4 MCP73831-2-OT

Commit message: final pcb?
Parts:
- removed C17: 0.1uF, Capacitor_SMD:C_0805_2012Metric_Pad1.18x1.45mm_HandSolder, symbol Device:C
- removed Q1: DMG2305UX-7, DMG2305UX-7:SOT91P240X110-3N_DMG2305UX-7, symbol DMG2305UX-7:DMG2305UX-7
- removed R9: 10k, Resistor_SMD:R_0805_2012Metric_Pad1.20x1.40mm_HandSolder, symbol Device:R
- added Q2: AO3400A, Package_TO_SOT_SMD:SOT-23, symbol Transistor_FET:AO3400A
- added R10, R11, R12: 1M, Resistor_SMD:R_0805_2012Metric_Pad1.20x1.40mm_HandSolder, symbol Device:R
- added R100: 100, Resistor_SMD:R_0805_2012Metric_Pad1.20x1.40mm_HandSolder, symbol Device:R
- R7: value 1k -> 2k
Connections:
- net LED_VCC is gone; now on net +BATT: C1.1, C2.1, C3.1, C4.1, C5.1, C6.1, C7.1, C8.1, D1.1 (VDD), D2.1 (VDD), D3.1 (VDD), D4.1 (VDD), D5.1 (VDD), D6.1 (VDD), D7.1 (VDD), D8.1 (VDD)
- net +BATT: now also R10.1
- net GND: now also Q2.2 (S), R12.2; no longer C1.2, C2.2, C3.2, C4.2, C5.2, C6.2, C7.2, C8.2, D1.3 (VSS), D2.3 (VSS), D3.3 (VSS), D4.3 (VSS), D5.3 (VSS), D6.3 (VSS), D7.3 (VSS), D8.3 (VSS)
- net IO7: now also R100.1
- net ADC: now reaches U1.18 (IO0)
- net ADC: now also R10.2, R11.1
- new net: Q2.1 (G), R100.2
- new net: R11.2, R12.1
- new net LED_GND: C1.2, C2.2, C3.2, C4.2, C5.2, C6.2, C7.2, C8.2, D1.3 (VSS), D2.3 (VSS), D3.3 (VSS), D4.3 (VSS), D5.3 (VSS), D6.3 (VSS), D7.3 (VSS), D8.3 (VSS), Q2.3 (D)
- no-connect marks 11 -> 10
