File: hardware/OHBeacon/OHBeacon.kicad_sch (KiCad schematic)
At the start: 51 parts, among them J1 Conn_01x01_Pin, J2 Conn_01x01_Pin, J3 Conn_01x01_Pin, J4 Conn_01x01_Pin, J5 USB_C_Receptacle_PowerOnly_6P, J6 Conn_01x04_Socket, P1 S2B-ZR-SM4A-TF, Q2 AO3400A, SW1 EN, SW2 I09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

Commit message: even more final PCB???
Parts:
- added R13: 500, Resistor_SMD:R_0805_2012Metric_Pad1.20x1.40mm_HandSolder, symbol Device:R
- added R9: 100k, Resistor_SMD:R_0805_2012Metric_Pad1.20x1.40mm_HandSolder, symbol Device:R
Connections:
- net DIN: now also R13.1; no longer U1.15 (IO3)
- net GND: now also R9.1
- net at Q2.1 (G), R100.2: now also R9.2
- new net: R13.2, U1.15 (IO3)
Other:
- moved on the sheet: C1, R100
